File: Hardware/SparkFun_GNSS_ZED-X20P.kicad_pcb (KiCad board)
At the start: 4 copper layers, 43.2 x 43.2 mm, 142 parts, among them J1 USB_C_Receptacle, J10 U.FL, J11 Conn_01x06, J2 Conn_01x06, J3 Conn_01x09, J4 Qwiic_RA, J5 SMA_Edge, J7 Qwiic_RA, J8 JST_Locking_4, J9 I2C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

Commit message: Post airwire review
Parts:
- removed D11: DF5A5.6LFU, SparkFun-Semiconductor-Standard:SOT-353
- removed JP6: UFL, SparkFun-Jumper:Jumper_2_NO_NoSilk
- removed R10: 0, SparkFun-Resistor:R_0402_1005Metric
- removed kibuzzard-66CAA7D2: G***, kibuzzard-66CAA7D2
- removed kibuzzard-6797CE44: G***, kibuzzard-6797CE44
- removed kibuzzard-6797D054: G***, kibuzzard-6797D054
- removed kibuzzard-6797D1F5: G***, kibuzzard-6797D1F5
- removed kibuzzard-6797D23B: G***, kibuzzard-6797D23B
- removed kibuzzard-6797D243: G***, kibuzzard-6797D243
- removed kibuzzard-6797D24B: G***, kibuzzard-6797D24B
- removed kibuzzard-67EC5731: G***, kibuzzard-67EC5731
- removed kibuzzard-67EC5C0F: G***, kibuzzard-67EC5C0F
- added D14: PESD0402, SparkFun-Capacitor:C_0402_1005Metric, F.Cu at (173.4, 105.1)
- added JP1: RF, SparkFun-Jumper:Jumper_3_NC-1_Trace, F.Cu at (171.8, 101.9)
- added L2: 33nH, SparkFun-Capacitor:C_0603_1608Metric, F.Cu at (171.1, 104.5)
- added kibuzzard-67ED93D1: G***, kibuzzard-67ED93D1, F.Cu at (173.4, 101.9)
- added kibuzzard-67ED9A28: G***, kibuzzard-67ED9A28, F.Cu at (169.5, 78.1)
- added kibuzzard-67ED9A4D: G***, kibuzzard-67ED9A4D, F.Cu at (154.3, 77.8)
- added kibuzzard-67ED9A5A: G***, kibuzzard-67ED9A5A, F.Cu at (164.5, 77.9)
- added kibuzzard-67ED9A5D: G***, kibuzzard-67ED9A5D, F.Cu at (167.0, 77.9)
- added kibuzzard-67ED9A70: G***, kibuzzard-67ED9A70, F.Cu at (161.9, 78.1)
- added kibuzzard-67ED9C3D: G***, kibuzzard-67ED9C3D, B.Cu at (145.9, 90.8)
- added kibuzzard-67ED9D32: G***, kibuzzard-67ED9D32, B.Cu at (160.7, 97.8)
- added kibuzzard-67ED9ED8: G***, kibuzzard-67ED9ED8, F.Cu at (169.5, 114.3)
- F1: value 6V/0.75A/1.5A -> 6V/0.5A/1A; footprint SparkFun-Fuse:1206 -> SparkFun-Fuse:0805
- R6: footprint SparkFun-Resistor:R_0402_1005Metric -> SparkFun-Resistor:R_0603_1608Metric
- moved D10 31.5 mm to (168.3, 81.3), turned to -90 degrees
- moved D13 14.0 mm to (153.0, 110.2), turned to -90 degrees
- moved C1 12.8 mm to (146.1, 95.9), turned to 90 degrees
- moved C3 10.5 mm to (171.1, 106.0), turned to 0 degrees
- moved D6 10.2 mm to (144.8, 100.3)
- moved C7 7.96 mm to (144.8, 102.2), turned to 0 degrees
- moved kibuzzard-6501FDDA 7.11 mm to (148.6, 89.5)
- moved kibuzzard-6797D04A 6.99 mm to (145.9, 85.7)
- moved kibuzzard-6797D04F 6.99 mm to (145.9, 88.3)
- moved J2 6.98 mm to (143.5, 83.2)
- moved kibuzzard-6797D058 6.98 mm to (145.7, 95.9)
- moved R12 6.79 mm to (144.8, 110.5), turned to 180 degrees
- moved kibuzzard-66CB829C 6.67 mm to (138.7, 89.5)
- moved F1 6.38 mm to (144.8, 98.4), turned to 180 degrees
- moved U2 6.24 mm to (148.9, 99.4), turned to 0 degrees
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Connections:
- D10 pad 4: 3.3V -> RX1/PICO
- D10 pad 5: unconnected-(D10-K4-Pad5) -> SDA/~{CS}
- D3 pad 2: RF_IN -> Net-(D3-A2)
- D6 pad 1: 5V -> Net-(D6-K)
- D6 pad 2: VBUS -> VUSB
- D7 pad 1: 5V -> Net-(D6-K)
- D8 pad 4: SDA/~{CS} -> 3.3V
- D8 pad 5: RX1/PICO -> V_BCKP
- F1 pad 1: VUSB -> 5V
- F1 pad 2: Net-(F1-Pad2) -> Net-(D6-K)
- J1 pad VBUS: Net-(F1-Pad2) -> VUSB
- J5 pad 1: Net-(J5-In) -> Net-(D3-A2)
- L1 pad 1: RF_IN -> Net-(D3-A2)
- U1 pad 1: unconnected-(U1-I/O1-Pad1) -> USB_D+
- U1 pad 3: unconnected-(U1-I/O2-Pad3) -> USB_D-
- U5 pad 38: VUSB -> 3.3V
Routing:
- net Net-(C3-Pad1): track 0.00 -> 10.3 mm, vias 0 -> 2
- net Net-(D3-A2): track 0.00 -> 7.13 mm
- net Net-(D14-A2): track 0.00 -> 4.49 mm
- net RF_IN: track 0.00 -> 3.67 mm
- net VCC_RF: track 0.00 -> 2.24 mm

Commit message: Update to v9.
Parts:
- U5: footprint SparkFun-GPS:ZED-F9 -> SparkFun-GPS:ZED-F9P_F9T_F9R_X20P
- moved kibuzzard-6797CF40 0.32 mm to (141.9, 89.5)
- moved J8 0.32 mm to (138.4, 89.5)
- turned JP4 to -90 degrees
- turned R12 to 0 degrees
- turned R13 to 0 degrees
- turned R9 to 180 degrees
Connections:
- D10 pad 3: SCL/SCK -> RX1/PICO
- D10 pad 4: RX1/PICO -> SDA/~{CS}
- D10 pad 5: SDA/~{CS} -> SCL/SCK
- D12 pad 1: PPS -> ~{RESET}
- D12 pad 3: ~{RESET} -> PPS
- D8 pad 1: TX2 -> RX2
- D8 pad 3: RX2 -> TX2
Routing:
- net SDA/~{CS}: track 0.00 -> 100.4 mm, vias 0 -> 3
- net SCL/SCK: track 0.00 -> 94.5 mm, vias 0 -> 3
- net GEO_STAT: track 0.00 -> 71.1 mm, vias 0 -> 3
- net RTK_STAT: track 0.00 -> 67.4 mm, vias 0 -> 3
- net RX2: track 0.00 -> 58.5 mm, vias 0 -> 1
- net TX1/POCI: track 0.00 -> 48.2 mm, vias 0 -> 2
- net RX1/PICO: track 0.00 -> 46.9 mm, vias 0 -> 1
- net TX2: track 0.00 -> 45.8 mm, vias 0 -> 2
- net PPS: track 0.00 -> 43.4 mm, vias 0 -> 1
- net 3V3_EN: track 0.00 -> 36.7 mm, vias 0 -> 2
- net 3.3V: track 0.00 -> 36.2 mm, vias 0 -> 8
- net V_BCKP: track 0.00 -> 26.9 mm, vias 0 -> 2
- net ~{RESET}: track 0.00 -> 23.5 mm, vias 0 -> 1
- net Net-(D6-K): track 0.00 -> 23.4 mm
- net 5V: track 0.00 -> 21.6 mm, vias 0 -> 1
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
Commit message: Add panel
Parts:
- removed kibuzzard-67EC5586: G***, kibuzzard-67EC5586
- removed kibuzzard-67EC5590: G***, kibuzzard-67EC5590
- removed kibuzzard-67EC559E: G***, kibuzzard-67EC559E
- removed kibuzzard-67EC55A8: G***, kibuzzard-67EC55A8
- added TP2: 1.0mm, SparkFun-Connector:TestPoint-1.0mm, B.Cu at (151.1, 89.2)
- added kibuzzard-680A9713: G***, kibuzzard-680A9713, B.Cu at (170.2, 86.2)
- added kibuzzard-680A971A: G***, kibuzzard-680A971A, B.Cu at (172.4, 86.0)
- added kibuzzard-680A9725: G***, kibuzzard-680A9725, B.Cu at (174.6, 86.0)
- added kibuzzard-680A972D: G***, kibuzzard-680A972D, B.Cu at (176.8, 86.8)
- L1, L2: value 33nH -> 47nH
- moved kibuzzard-66CB82FB 5.08 mm to (140.7, 87.0)
- moved kibuzzard-66CB830B 4.92 mm to (140.7, 92.1)
Connections:
- D9 pad 1: GND -> GEO_STAT
- JP8 pad 2: GEO_STAT -> 3.3V
- U5 pad 10: (no net) -> unconnected-(U5-NC-Pad10)
- U5 pad 11: (no net) -> unconnected-(U5-NC-Pad11)
- U5 pad 13: (no net) -> unconnected-(U5-NC-Pad13)
- U5 pad 15: (no net) -> unconnected-(U5-NC-Pad15)
- U5 pad 16: (no net) -> unconnected-(U5-NC-Pad16)
- U5 pad 17: (no net) -> unconnected-(U5-NC-Pad17)
- U5 pad 18: (no net) -> unconnected-(U5-NC-Pad18)
- U5 pad 21: (no net) -> unconnected-(U5-NC-Pad21)
- U5 pad 22: (no net) -> unconnected-(U5-NC-Pad22)
- U5 pad 23: (no net) -> unconnected-(U5-NC-Pad23)
- U5 pad 24: (no net) -> unconnected-(U5-NC-Pad24)
- U5 pad 25: (no net) -> unconnected-(U5-NC-Pad25)
- U5 pad 28: (no net) -> unconnected-(U5-NC-Pad28)
- U5 pad 29: (no net) -> unconnected-(U5-NC-Pad29)
- U5 pad 30: (no net) -> unconnected-(U5-NC-Pad30)
- U5 pad 31: (no net) -> unconnected-(U5-NC-Pad31)
- U5 pad 35: (no net) -> unconnected-(U5-NC-Pad35)
- U5 pad 52: (no net) -> unconnected-(U5-NC-Pad52)
- U5 pad 54: (no net) -> unconnected-(U5-NC-Pad54)
- U5 pad 8: (no net) -> unconnected-(U5-NC-Pad8)
- U5 pad 9: (no net) -> unconnected-(U5-NC-Pad9)
Routing:
- net 3.3V: track 36.2 -> 41.6 mm, vias 8 -> 9
- net GEO_STAT: track 71.1 -> 76.0 mm, vias 3 -> 4
- net SCL/SCK: track 94.5 -> 97.9 mm
- net V_BCKP: track 26.9 -> 28.3 mm
- net TX1/POCI: track 48.2 -> 49.0 mm
- net PPS: track 43.4 -> 42.6 mm
- net GND: vias 108 -> 112
