File: Hardware/SparkFun_GNSS_ZED-X20P.kicad_pcb (KiCad board)
At the start: 4 copper layers, 43.2 x 43.2 mm, 143 parts, among them J1 USB_C_Receptacle, J10 U.FL, J11 Conn_01x06, J2 Conn_01x06, J3 Conn_01x09, J4 Qwiic_RA, J5 SMA_Edge, J7 Qwiic_RA, J8 JST_Locking_4, J9 I2C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

Commit message: Update to new symbol/fp locations
Parts:
- J10: value U.FL -> Val**
- J11, J2: footprint SparkFun-Connector:1x06 -> SparkFun-Connector:1x06_P2.54mm
- J3: footprint SparkFun-Connector:1x09 -> SparkFun-Connector:1x09_P2.54mm
- J4, J7: footprint SparkFun-Connector:JST_SMD_1.0mm-4_Black -> SparkFun-Connector:JST_1x04_P1.0mm_Horizontal_SMD
- J5: footprint SparkFun-Connector:SMA_Edge -> SparkFun-Connector:SMA_Edge_8mm
- J8: footprint SparkFun-Connector:JST_SMD_1.25mm-4_Locking -> SparkFun-Connector:JST_1x04_P1.25mm_Locking_Horizontal_SMD
- J9: footprint SparkFun-Connector:1x04 -> SparkFun-Connector:1x04_P2.54mm
- U5: footprint SparkFun-GPS:ZED-F9P_F9T_F9R_X20P -> SparkFun-GNSS:ZED-F9P_F9T_F9R_X20P
